File: h8read.kicad_pcb (KiCad board)
At the start: 2 copper layers, 47.2 x 46.7 mm, 11 parts, among them U1 27C010, U2 H8/3664F FP-64E QFP64P0.8

Commit message: r1 gerbers
Parts:
- added C3: 22p XTAL, Capacitor_SMD:C_0805_2012Metric_Pad1.18x1.45mm_HandSolder, F.Cu at (137.9, 81.4)
- added C4: 20p XTAL, Capacitor_SMD:C_0805_2012Metric_Pad1.18x1.45mm_HandSolder, F.Cu at (134.7, 77.0)
- added H1: MountingHole, MountingHole:MountingHole_2.7mm_M2.5_DIN965, F.Cu at (142.9, 73.7)
- added H2: MountingHole, MountingHole:MountingHole_2.7mm_M2.5_DIN965, F.Cu at (142.9, 112.4)
- added R1: A16, Resistor_SMD:R_1206_3216Metric_Pad1.30x1.75mm_HandSolder, F.Cu at (116.2, 77.5)
- added TP1: XTAL, TestPoint:TestPoint_Pad_1.0x1.0mm, F.Cu at (134.7, 85.2)
- added Y1: 8MHz, Crystal:Crystal_SMD_5032-4Pin_5.0x3.2mm, F.Cu at (134.7, 80.9)
- C1, C2: value 1uF PWR -> PWR
- JP5: value X1 -> ~{RES}
- JP6: value ~{NMI} -> TEST
- JP7: value TEST -> ~{NMI}
- moved JP7 25.7 mm to (117.9, 98.4), turned to 0 degrees
- moved JP6 24.2 mm to (140.2, 89.3), turned to 180 degrees
- moved JP5 3.06 mm to (140.2, 92.3)
- moved C2 2.44 mm to (130.2, 79.1)
- moved C1 2.33 mm to (139.6, 86.0), turned to 180 degrees
Connections:
- U1 pad 2: unconnected-(U1-A16-Pad2) -> Net-(U1-A16)
- U2 pad 10: unconnected-(U2-OSC1-Pad10) -> OSC1
- U2 pad 11: unconnected-(U2-OSC2-Pad11) -> OSC2
- U2 pad 35: Net-(JP6-B) -> Net-(JP7-B)
- U2 pad 5: Net-(JP5-B) -> GND
- U2 pad 7: unconnected-(U2-~{RES}-Pad7) -> Net-(JP5-B)
- U2 pad 8: Net-(JP7-B) -> Net-(JP6-B)
Routing:
- net GND: track 56.9 -> 35.9 mm, vias 62 -> 70
- net Net-(U1-A16): track 0.00 -> 11.0 mm
- net OSC2: track 0.00 -> 10.5 mm
- net OSC1: track 0.00 -> 8.76 mm
- net VCC: track 151.8 -> 160.4 mm, vias 8 -> 7
- net A6: track 38.0 -> 30.0 mm
- net ~{WE}: track 43.8 -> 35.9 mm
- net Net-(JP6-B): track 5.38 -> 12.1 mm
- net Net-(JP5-B): track 5.42 -> 11.4 mm
- net Net-(JP7-B): track 8.76 -> 5.32 mm
- net unconnected-(U2-~{RES}-Pad7): track 3.33 -> 0.00 mm, vias 1 -> 0
- net A1: track 35.4 -> 36.5 mm
- net A2: track 36.8 -> 37.6 mm
- net A11: track 13.7 -> 14.3 mm
Other:
- board text added: "!"
- board text added: "Keep clear"

Commit message: second revision
Parts:
- added J1: PWR, Connector_PinHeader_2.54mm:PinHeader_1x02_P2.54mm_Vertical, F.Cu at (120.8, 75.9)
Routing:
- net GND: track 35.9 -> 45.2 mm
- net VCC: track 160.4 -> 163.2 mm, vias 7 -> 5
- net Net-(U2-VCL): vias 1 -> 0
- added copper zone on B.Cu, net VCC
- added copper zone on F.Cu, net VCC
Other:
- board size 47.2 x 46.7 mm -> 47.2 x 46.5 mm
