File: h8read.kicad_sch (KiCad schematic)
At the start: 11 parts, among them U1 27C010, U2 H8/3664F FP-64E QFP64P0.8

Commit message: r1 gerbers
Parts:
- added C3: 22p XTAL, Capacitor_SMD:C_0805_2012Metric_Pad1.18x1.45mm_HandSolder, symbol Device:C_Small
- added C4: 20p XTAL, Capacitor_SMD:C_0805_2012Metric_Pad1.18x1.45mm_HandSolder, symbol Device:C_Small
- added H1, H2: MountingHole, MountingHole:MountingHole_2.7mm_M2.5_DIN965, symbol Mechanical:MountingHole
- added R1: A16, Resistor_SMD:R_1206_3216Metric_Pad1.30x1.75mm_HandSolder, symbol Device:R_Small
- added TP1: XTAL, TestPoint:TestPoint_Pad_1.0x1.0mm, symbol Connector:TestPoint_Probe
- added Y1: 8MHz, Crystal:Crystal_SMD_5032-4Pin_5.0x3.2mm, symbol Device:Crystal_GND24_Small
- JP5: value X1 -> ~{RES}
- JP6: value ~{NMI} -> TEST
- JP7: value TEST -> ~{NMI}
Connections:
- net GND: now also U2.5 (X1), C3.1, C4.2
- net VCC: now also R1.2
- net at JP5.2 (B): now also U2.7 (~{RES}); no longer U2.5 (X1)
- net at U1.2 (A16): now also R1.1
- net at U2.8 (TEST): now also JP6.2 (B); no longer JP7.2 (B)
- net OSC1: now reaches U2.10 (OSC1)
- net OSC1: now also C3.2, TP1.1, Y1.1
- net OSC2: now reaches U2.11 (OSC2)
- net OSC2: now also C4.1, Y1.3
- net at U2.35 (~{NMI}): now also JP7.2 (B); no longer JP6.2 (B)
- no-connect marks 2 -> 4
Other:
- moved on the sheet: C102

Commit message: second revision
Parts:
- added J1: PWR, Connector_PinHeader_2.54mm:PinHeader_1x02_P2.54mm_Vertical, symbol Connector:Conn_01x02_Pin
- C102: value 1uF PWR -> PWR
Connections:
- net GND: now also J1.2 (Pin_2)
- net VCC: now also J1.1 (Pin_1)
Changed lines of the file:
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@@
+    )
+  )
+  (global_label "GND" (shape passive) (at 102.87 134.62 0) (fields_autoplaced)
+    (effects (font (size 1.27 1.27)) (justify left))
+    (property "Intersheetrefs" "${INTERSHEET_REFS}" (at 108.6144 134.62 0)
+      (effects (font (size 1.27 1.27)) (justify left) hide)
+    )
+    (property "Netclass" "PWR" (at 102.87 136.8108 0)
+      (effects (font (size 1.27 1.27)) (justify left) hide)
     )
   )
@@
     (property "Intersheetrefs" "${INTERSHEET_REFS}" (at 154.0993 83.7406 0)
       (effects (font (size 1.27 1.27)) (justify right) hide)
+    )
+  )
+  (global_label "VCC" (shape passive) (at 102.87 132.08 0) (fields_autoplaced)
+    (effects (font (size 1.27 1.27)) (justify left))
+    (property "Intersheetrefs" "${INTERSHEET_REFS}" (at 108.3725 132.08 0)
+      (effects (font (size 1.27 1.27)) (justify left) hide)
+    )
+    (property "Netclass" "PWR" (at 102.87 134.2708 0)
+      (effects (font (size 1.27 1.27)) (justify left) hide)
     )
   )
@@
       (effects (font (size 1.27 1.27)))
     )
-    (property "Value" "1uF PWR" (at 100.3362 118.11 0)
+    (property "Value" "PWR" (at 100.3362 118.11 0)
       (effects (font (size 1.27 1.27)) (justify left) hide)
     )
@@
     )
   )
+  (symbol (lib_id "Connector:Conn_01x02_Pin") (at 97.79 132.08 0) (unit 1)
+    (in_bom yes) (on_board yes) (dnp no) (fields_autoplaced)
+    (property "Reference" "J1" (at 98.425 127 0)
+      (effects (font (size 1.27 1.27)))
+    )
+    (property "Value" "PWR" (at 98.425 129.54 0)
+      (effects (font (size 1.27 1.27)))
+    )
+    (property "Footprint" "Connector_PinHeader_2.54mm:PinHeader_1x02_P2.54mm_Vertical" (at 97.79 132.08 0)
+      (effects (font (size 1.27 1.27)) hide)
+    )
+    (property "Datasheet" "~" (at 97.79 132.08 0)
+      (effects (font (size 1.27 1.27)) hide)
+    )
+    (pin "1")
+    (pin "2")
+    (instances
+      (project "h8read"
+        (path "/773aad54-fe8c-42bc-859d-878858927827"
+          (reference "J1") (unit 1)
+        )
+      )
+    )
+  )
   (symbol (lib_id "Device:C_Small") (at 143.51 120.65 180) (unit 1)
     (in_bom yes) (on_board yes) (dnp no) (fields_autoplaced)
@@
       (effects (font (size 1.27 1.27)) (justify right))
     )
-    (property "Value" "1uF PWR" (at 140.97 119.3738 0)
-      (effects (font (size 1.27 1.27)) (justify left) hide)
-    )
+    (property "Value" "PWR" (at 140.97 119.3738 0)
+      (effects (font (size 1.27 1.27)) (justify left) hide)
+    )
